Commit message: corrected bug in motcontrol updated launchfiles updated tags config updated Bacon

File: src/sandwich/urdf/sandwich.urdf (robot description, URDF)
Before this commit: robot sandwich, 3 links, 2 joints
Links:
- added link batt_link; visual box size=0.19 0.09 0.03
- added link camera; visual cylinder length=0.01 radius=0.01
- link base_link: geometry 
- link left_wheel: geometry visual cylinder length=0.005 radius=0.035
- link right_wheel: geometry visual cylinder length=0.005 radius=0.035
Joints:
- added joint base_link_to_batt_link: type fixed, parent base_link, child batt_link, origin xyz=0.045 0.0 0.025
- added joint base_link_to_camera: type fixed, parent base_link, child camera, origin xyz=0.145 0.0 0.041 rpy=-1.57 0.0 -1.57
- joint base_link_to_left_wheel: origin xyz=-0.045 0.05 -0.025 -> xyz=0.0 0.05 0.0
- joint base_link_to_right_wheel: origin xyz=-0.045 -0.05 -0.025 -> xyz=0.0 -0.05 0.0
